Commit message: Added files for adding multi realsense d435 on ridgeback-yumi

File: ridgeback_yumi_description/urdf/ridgeback_yumi.urdf.xacro (robot description, xacro)
@@ -36,6 +36,15 @@
   <xacro:property name="yumi_offset_x" value="0.06" />
   <xacro:property name="yumi_height" value="0.25" />
-  <xacro:property name="kinect_zrotation_fix" value="${- PI / 2.0}" />
-  <xacro:property name="kinect_base_pitch" value="${ -PI/2.0 }" />
+  <!-- Constants for Intel d435 mount dimensions -->
+  <!-- Constants for robot dimensions -->
+  <xacro:property name="mass" value="0.5" /> <!-- arbitrary value for mass -->
+  <xacro:property name="width" value="0.065" /> <!-- Radius of the camera mount -->
+  <xacro:property name="height" value="0.4" /> <!--Height of the camera mount -->
+  <xacro:property name="camera_length" value="0.09" /> <!-- Size of square 'camera' box -->
+  <xacro:property name="camera_width" value="0.025" /> <!-- Space btw top of beam and the each joint -->
+  <xacro:property name="angle_diff" value="${pi/3}" /> <!-- Space btw top of beam and the each joint -->
+  <xacro:property name="angle_tilt_1" value="${pi/6}" /> <!-- Space btw top of beam and the each joint -->
+  <xacro:property name="angle_tilt_2" value="${pi/36}" /> <!-- Space btw top of beam and the each joint -->
+  <xacro:property name="angle_tilt_3" value="${pi/36}" /> <!-- Space btw top of beam and the each joint -->
   <joint name="ridgeback_base_to_pedestal" type="fixed">
     <origin rpy="0 0 ${PI}" xyz="${pedestal_offset_x} 0 ${pedestal_height}" />
@@ -64,59 +73,131 @@
     <child link="yumi_base_link" />
   </joint>
-  <link name="kinect2">
-    <visual>
-      <origin xyz="0 0 0" rpy="0 0 0" />
-      <geometry>
-        <mesh scale="0.001 0.001 0.001" filename="package://yumi_description/meshes/accesories/KinectXboxOne.stl"/>
-      </geometry>
-      <material name="Black" />
-    </visual>
-  </link>
-  <link name="left_kinect_base">
-      <visual>
-        <origin xyz="0 0 0" rpy="0 0 0" />
-        <geometry>
-          <box size="0.4 0.02 0.02" />
-        </geometry>
-        <material name="Grey" />
-      </visual>
-  </link>
-  <link name="right_kinect_base">
-      <visual>
-        <origin xyz="0 0 0" rpy="0 0 0" />
-        <geometry>
-          <box size="0.4 0.02 0.02" />
-        </geometry>
-        <material name="Grey" />
-      </visual>
-  </link>
-  <link name="middle_kinect_base">
-      <visual>
-        <origin xyz="0 0 0" rpy="0 0 0" />
-        <geometry>
-          <box size="0.4 0.02 0.02" />
-        </geometry>
-        <material name="Grey" />
-      </visual>
-  </link>
-   <joint name="kinect2_to_right_kinect_base" type="fixed">
+  <xacro:include filename="$(find multi_d435_description)/urdf/multi_d435.gazebo" />
+  <joint name="yumi_to_mount" type="fixed">
     <parent link="yumi_base_link" />
-    <child link="right_kinect_base" />
-    <origin rpy="0 ${-PI/2} 0.17" xyz="-0.1 -0.03 0.56" />
-  </joint>
-  <joint name="kinect2_to_left_kinect_base" type="fixed">
-    <parent link="yumi_base_link" />
-    <child link="left_kinect_base" />
-    <origin rpy="0 ${-PI/2} -0.17" xyz="-0.1 0.03 0.56" />
-  </joint>
-  <joint name="yumi_to_middle_kinect_base" type="fixed">
-    <parent link="yumi_base_link" />
-    <child link="middle_kinect_base" />
-    <origin rpy="0 ${kinect_base_pitch} 0" xyz="-0.1 0 0.56" />
-  </joint>
-  <joint name="middle_kinect_base_to_kinect2" type="fixed">
-    <parent link="middle_kinect_base" />
-    <child link="kinect2" />
-    <origin rpy="${-PI/2} 0 ${kinect_zrotation_fix}" xyz="0.25 0 0" />
-  </joint>
+    <child link="multi_d435_mount" />
+    <origin rpy="0 0 0" xyz="-0.05 0 0.4" />
+  </joint>
+  <!-- Camera mount Link -->
+  <link name="multi_d435_mount">
+    <collision>
+      <origin xyz="0 0 ${height/2}" rpy="0 0 0"/>
+      <geometry>
+         <cylinder radius="${width}" length="${height}"/>
+      </geometry>
+    </collision>
+   <visual>
+      <origin xyz="0 0 0" rpy="0 0 ${pi/6}"/>
+      <geometry>
+	       <mesh scale= "0.007 0.007 0.01" filename="package://multi_d435_description/meshes/d435_mount.dae"/>
+      </geometry>
+    </visual>
+    <inertial>
+      <origin xyz="0 0 ${height/2}" rpy="0 0 0"/>
+      <mass value="${mass}"/>
+      <inertia
+	  ixx="${mass / 12.0 * (width*width + height*height)}" ixy="0.0" ixz="0.0"
+	  iyy="${mass / 12.0 * (height*height + width*width)}" iyz="0.0"
+	  izz="${mass / 12.0 * (width*width + width*width)}"/>
+    </inertial>
+  </link>
+  <joint name="camera_joint_1" type="fixed">
+    <origin xyz="${width+camera_width} 0 ${height-camera_length}" rpy="0 ${angle_tilt_1} 0"/>
+    <parent link="multi_d435_mount"/>
+    <child link="camera_link_1"/>
+  </joint>
+  <joint name="camera_joint_2" type="fixed">
+    <origin xyz="${(width+camera_width)*cos(angle_diff)} ${(width+camera_width)*sin(angle_diff)} ${height-camera_length}" rpy="0 ${angle_tilt_2} ${angle_diff}"/>
+    <parent link="multi_d435_mount"/>
+    <child link="camera_link_2"/>
+  </joint>
+  <joint name="camera_joint_3" type="fixed">
+    <origin xyz="${(width+camera_width)*cos(angle_diff)} -${(width+camera_width)*sin(angle_diff)} ${height-camera_length}" rpy="0 ${angle_tilt_3} -${angle_diff}"/>
+    <parent link="multi_d435_mount"/>
+    <child link="camera_link_3"/>
+  </joint>
+  <!-- Camera 1-->
+  <link name="camera_link_1">
+    <collision>
+      <origin xyz="0 0 0" rpy="0 0 0"/>
+      <geometry>
+	       <box size="${camera_length} ${camera_width} ${camera_width}"/>
+      </geometry>
+    </collision>
+    <visual>
+      <origin xyz="0 0 0" rpy="${pi/2} ${pi/2} ${pi/2}"/>
+      <geometry>
+	       <mesh filename="package://multi_d435_description/meshes/d435.dae"/>
+      </geometry>
+      <material name="red"/>
+    </visual>
+    <inertial>
+      <mass value="0.0615752" />
+      <origin xyz="0 0 0" rpy="0 0 0"/>
+      <inertia ixx="9.108e-05" ixy="0" ixz="0" iyy="2.51e-06" iyz="0" izz="8.931e-05" />
+    </inertial>
+  </link>
+  <!-- Camera 2-->
+  <link name="camera_link_2">
+    <collision>
+      <origin xyz="0 0 0" rpy="0 0 0"/>
+      <geometry>
+	       <box size="${camera_length} ${camera_width} ${camera_width}"/>
+      </geometry>
+    </collision>
+    <visual>
+      <origin xyz="0 0 0" rpy="${pi/2} ${pi/2} ${pi/2}"/>
+      <geometry>
+	       <mesh filename="package://multi_d435_description/meshes/d435.dae"/>
+      </geometry>
+      <material name="red"/>
+    </visual>
+    <inertial>
+      <mass value="0.0615752" />
+      <origin xyz="0 0 0" rpy="0 0 0"/>
+      <inertia ixx="9.108e-05" ixy="0" ixz="0" iyy="2.51e-06" iyz="0" izz="8.931e-05" />
+    </inertial>
+  </link>
+  <!-- Camera 3-->
+  <link name="camera_link_3">
+    <collision>
+      <origin xyz="0 0 0" rpy="0 0 0"/>
+      <geometry>
+	       <box size="${camera_length} ${camera_width} ${camera_width}"/>
+      </geometry>
+    </collision>
+    <visual>
+      <origin xyz="0 0 0" rpy="${pi/2} ${pi/2} ${pi/2}"/>
+      <geometry>
+	       <mesh filename="package://multi_d435_description/meshes/d435.dae"/>
+      </geometry>
+      <material name="red"/>
+    </visual>
+    <inertial>
+      <mass value="0.0615752" />
+      <origin xyz="0 0 0" rpy="0 0 0"/>
+      <inertia ixx="9.108e-05" ixy="0" ixz="0" iyy="2.51e-06" iyz="0" izz="8.931e-05" />
+    </inertial>
+  </link>
+  <joint name="camera_optical_joint_1" type="fixed">
+    <origin xyz="0 0 0" rpy="${-pi/2} 0 ${-pi/2}"/>
+    <parent link="camera_link_1"/>
+    <child link="camera_link_optical_1"/>
+  </joint>
+  <link name="camera_link_optical_1">
+  </link>
+  <joint name="camera_optical_joint_2" type="fixed">
+    <origin xyz="0 0 0" rpy="${-pi/2} 0 ${-pi/2}"/>
+    <parent link="camera_link_2"/>
+    <child link="camera_link_optical_2"/>
+  </joint>
+  <link name="camera_link_optical_2">
+  </link>
+  <joint name="camera_optical_joint_3" type="fixed">
+    <origin xyz="0 0 0" rpy="${-pi/2} 0 ${-pi/2}"/>
+    <parent link="camera_link_3"/>
+    <child link="camera_link_optical_3"/>
+  </joint>
+  <link name="camera_link_optical_3">
+  </link>
 </robot>

Commit message: Modified URDF with double mount multi-inteld435 cameras

File: ridgeback_yumi_description/urdf/ridgeback_yumi.urdf.xacro (robot description, xacro)
@@ -36,15 +36,4 @@
   <xacro:property name="yumi_offset_x" value="0.06" />
   <xacro:property name="yumi_height" value="0.25" />
-  <!-- Constants for Intel d435 mount dimensions -->
-  <!-- Constants for robot dimensions -->
-  <xacro:property name="mass" value="0.5" /> <!-- arbitrary value for mass -->
-  <xacro:property name="width" value="0.065" /> <!-- Radius of the camera mount -->
-  <xacro:property name="height" value="0.4" /> <!--Height of the camera mount -->
-  <xacro:property name="camera_length" value="0.09" /> <!-- Size of square 'camera' box -->
-  <xacro:property name="camera_width" value="0.025" /> <!-- Space btw top of beam and the each joint -->
-  <xacro:property name="angle_diff" value="${pi/3}" /> <!-- Space btw top of beam and the each joint -->
-  <xacro:property name="angle_tilt_1" value="${pi/6}" /> <!-- Space btw top of beam and the each joint -->
-  <xacro:property name="angle_tilt_2" value="${pi/36}" /> <!-- Space btw top of beam and the each joint -->
-  <xacro:property name="angle_tilt_3" value="${pi/36}" /> <!-- Space btw top of beam and the each joint -->
   <joint name="ridgeback_base_to_pedestal" type="fixed">
     <origin rpy="0 0 ${PI}" xyz="${pedestal_offset_x} 0 ${pedestal_height}" />
@@ -73,131 +62,186 @@
     <child link="yumi_base_link" />
   </joint>
-  <xacro:include filename="$(find multi_d435_description)/urdf/multi_d435.gazebo" />
-  <joint name="yumi_to_mount" type="fixed">
-    <parent link="yumi_base_link" />
-    <child link="multi_d435_mount" />
-    <origin rpy="0 0 0" xyz="-0.05 0 0.4" />
-  </joint>
-  <!-- Camera mount Link -->
-  <link name="multi_d435_mount">
-    <collision>
-      <origin xyz="0 0 ${height/2}" rpy="0 0 0"/>
-      <geometry>
-         <cylinder radius="${width}" length="${height}"/>
-      </geometry>
-    </collision>
-   <visual>
-      <origin xyz="0 0 0" rpy="0 0 ${pi/6}"/>
-      <geometry>
-	       <mesh scale= "0.007 0.007 0.01" filename="package://multi_d435_description/meshes/d435_mount.dae"/>
-      </geometry>
-    </visual>
-    <inertial>
-      <origin xyz="0 0 ${height/2}" rpy="0 0 0"/>
-      <mass value="${mass}"/>
-      <inertia
-	  ixx="${mass / 12.0 * (width*width + height*height)}" ixy="0.0" ixz="0.0"
-	  iyy="${mass / 12.0 * (height*height + width*width)}" iyz="0.0"
-	  izz="${mass / 12.0 * (width*width + width*width)}"/>
-    </inertial>
-  </link>
-  <joint name="camera_joint_1" type="fixed">
-    <origin xyz="${width+camera_width} 0 ${height-camera_length}" rpy="0 ${angle_tilt_1} 0"/>
-    <parent link="multi_d435_mount"/>
-    <child link="camera_link_1"/>
-  </joint>
-  <joint name="camera_joint_2" type="fixed">
-    <origin xyz="${(width+camera_width)*cos(angle_diff)} ${(width+camera_width)*sin(angle_diff)} ${height-camera_length}" rpy="0 ${angle_tilt_2} ${angle_diff}"/>
-    <parent link="multi_d435_mount"/>
-    <child link="camera_link_2"/>
-  </joint>
-  <joint name="camera_joint_3" type="fixed">
-    <origin xyz="${(width+camera_width)*cos(angle_diff)} -${(width+camera_width)*sin(angle_diff)} ${height-camera_length}" rpy="0 ${angle_tilt_3} -${angle_diff}"/>
-    <parent link="multi_d435_mount"/>
-    <child link="camera_link_3"/>
-  </joint>
-  <!-- Camera 1-->
-  <link name="camera_link_1">
-    <collision>
-      <origin xyz="0 0 0" rpy="0 0 0"/>
-      <geometry>
-	       <box size="${camera_length} ${camera_width} ${camera_width}"/>
-      </geometry>
-    </collision>
-    <visual>
-      <origin xyz="0 0 0" rpy="${pi/2} ${pi/2} ${pi/2}"/>
-      <geometry>
-	       <mesh filename="package://multi_d435_description/meshes/d435.dae"/>
-      </geometry>
-      <material name="red"/>
-    </visual>
-    <inertial>
-      <mass value="0.0615752" />
-      <origin xyz="0 0 0" rpy="0 0 0"/>
-      <inertia ixx="9.108e-05" ixy="0" ixz="0" iyy="2.51e-06" iyz="0" izz="8.931e-05" />
-    </inertial>
-  </link>
-  <!-- Camera 2-->
-  <link name="camera_link_2">
-    <collision>
-      <origin xyz="0 0 0" rpy="0 0 0"/>
-      <geometry>
-	       <box size="${camera_length} ${camera_width} ${camera_width}"/>
-      </geometry>
-    </collision>
-    <visual>
-      <origin xyz="0 0 0" rpy="${pi/2} ${pi/2} ${pi/2}"/>
-      <geometry>
-	       <mesh filename="package://multi_d435_description/meshes/d435.dae"/>
-      </geometry>
-      <material name="red"/>
-    </visual>
-    <inertial>
-      <mass value="0.0615752" />
-      <origin xyz="0 0 0" rpy="0 0 0"/>
-      <inertia ixx="9.108e-05" ixy="0" ixz="0" iyy="2.51e-06" iyz="0" izz="8.931e-05" />
-    </inertial>
-  </link>
-  <!-- Camera 3-->
-  <link name="camera_link_3">
-    <collision>
-      <origin xyz="0 0 0" rpy="0 0 0"/>
-      <geometry>
-	       <box size="${camera_length} ${camera_width} ${camera_width}"/>
-      </geometry>
-    </collision>
-    <visual>
-      <origin xyz="0 0 0" rpy="${pi/2} ${pi/2} ${pi/2}"/>
-      <geometry>
-	       <mesh filename="package://multi_d435_description/meshes/d435.dae"/>
-      </geometry>
-      <material name="red"/>
-    </visual>
-    <inertial>
-      <mass value="0.0615752" />
-      <origin xyz="0 0 0" rpy="0 0 0"/>
-      <inertia ixx="9.108e-05" ixy="0" ixz="0" iyy="2.51e-06" iyz="0" izz="8.931e-05" />
-    </inertial>
-  </link>
-  <joint name="camera_optical_joint_1" type="fixed">
+  <!-- Constants for Intel d435 mount dimensions -->
+  <!-- Constants for camera mount  dimensions -->
+   <xacro:property name="massp" value="0.05" /> <!-- mass for lower mount -->
+   <xacro:property name="widthp" value="0.025" /> <!-- width of lower mount -->
+   <xacro:property name="heightp" value="0.085" /> <!--height of lower mount -->
+   <xacro:property name="mass" value="0.05" /> <!-- mass for camera mount -->
+   <xacro:property name="width" value="0.02" /> <!-- radius of the camera mount -->
+   <xacro:property name="height" value="0.085" /> <!--height of the camera mount -->
+   <xacro:property name="camera_length" value="0.0492" /> <!-- Size of square 'camera' box -->
+   <xacro:property name="camera_width" value="0.025" /> <!-- Size of square 'camera' box -->
+   <xacro:property name="angle_diff" value="${pi/3}" /> <!-- angle btw camera mount -->
+   <xacro:property name="angle_tilt_1" value="0" /> <!-- horizontal tilt of camera 1  -->
+   <xacro:property name="angle_tilt_2" value="0" /> <!-- horizontal tilt of camera 2 -->
+   <xacro:property name="angle_tilt_3" value="0" /> <!-- horizontal tilt of camera 3 -->
+  <xacro:include filename="$(find ridgeback_yumi_description)/urdf/multi_d435.gazebo" />
+  <joint name="ridgeback_to_mount" type="fixed">
+    <parent link="mid_mount" />
+    <child link="mount_tripod" />
+    <origin rpy="0 0 0" xyz="0.17 0 0.72" />
+  </joint>
+   <!-- Tripod -->
+      <link name="mount_tripod">
+        <collision>
+          <origin xyz="0 0 ${heightp/2}" rpy="0 0 0"/>
+          <geometry>
+             <cylinder radius="${widthp}" length="${heightp}"/>
+          </geometry>
+        </collision>
+        <visual>
+          <origin xyz="0 0 0" rpy="${pi/2} 0 0"/>
+          <geometry>
+    	       <mesh filename="package://ridgeback_yumi_description/meshes/tripod_simplified.STL"/>
+          </geometry>
+          <material name="orange"/>
+        </visual>
+        <inertial>
+          <origin xyz="0 0 ${heightp/2}" rpy="0 0 0"/>
+          <mass value="${massp}"/>
+          <inertia
+    	  ixx="${massp / 12.0 * (widthp*widthp + heightp*heightp)}" ixy="0.0" ixz="0.0"
+    	  iyy="${massp / 12.0 * (heightp*heightp + widthp*widthp)}" iyz="0.0"
+    	  izz="${massp / 12.0 * (widthp*widthp + widthp*widthp)}"/>
+        </inertial>
+      </link>
+      <joint name="camera_mount_joint" type="fixed">
+        <parent link="mount_tripod" />
+        <child link="multi_d435_mount" />
+        <origin rpy="0 0 0" xyz="0 0 ${heightp} " />
+      </joint>
+      <!-- Camera mount Link -->
+      <link name="multi_d435_mount">
+        <collision>
+          <origin xyz="0 0 ${height/2}" rpy="0 0 0"/>
+          <geometry>
+             <cylinder radius="${width}" length="${height}"/>
+          </geometry>
+        </collision>
+       <visual>
+          <origin xyz="0 0 0" rpy="0 0 ${pi/6}"/>
+          <geometry>
+    	       <mesh filename="package://ridgeback_yumi_description/meshes/D435x6_mounting-support.STL"/>
+          </geometry>
+        </visual>
+        <inertial>
+          <origin xyz="0 0 ${height/2}" rpy="0 0 0"/>
+          <mass value="${mass}"/>
+          <inertia
+    	  ixx="${mass / 12.0 * (width*width + height*height)}" ixy="0.0" ixz="0.0"
+    	  iyy="${mass / 12.0 * (height*height + width*width)}" iyz="0.0"
+    	  izz="${mass / 12.0 * (width*width + width*width)}"/>
+        </inertial>
+      </link>
+      <joint name="camera_joint_1" type="fixed">
+        <origin xyz="${width+camera_width} 0 ${height-camera_length}" rpy="${pi/2} ${angle_tilt_1} 0"/>
+        <parent link="multi_d435_mount"/>
+        <child link="camera1_link"/>
+      </joint>
+      <joint name="camera_joint_2" type="fixed">
+        <origin xyz="${(width+camera_width)*cos(angle_diff)} ${(width+camera_width)*sin(angle_diff)} ${height-camera_length}" rpy="${pi/2} ${angle_tilt_2} ${angle_diff}"/>
+        <parent link="multi_d435_mount"/>
+        <child link="camera2_link"/>
+      </joint>
+      <joint name="camera_joint_3" type="fixed">
+        <origin xyz="${(width+camera_width)*cos(angle_diff)} -${(width+camera_width)*sin(angle_diff)} ${height-camera_length}" rpy="${pi/2} ${angle_tilt_3} -${angle_diff}"/>
+        <parent link="multi_d435_mount"/>
+        <child link="camera3_link"/>
+      </joint>
+      <!-- Camera 1-->
+      <link name="camera1_link">
+        <collision>
+          <origin xyz="0 0 0" rpy="0 0 0"/>
+          <geometry>
+    	       <box size="${camera_width} ${camera_length} ${camera_width}"/>
+          </geometry>
+        </collision>
+        <visual>
+          <origin xyz="0 0 0" rpy="${pi/2} 0 ${pi/2}"/>
+          <geometry>
+    	       <mesh filename="package://ridgeback_yumi_description/meshes/Intel_RealSense_Depth_Camera_D435.STL"/>
+          </geometry>
+          <material name="red"/>
+        </visual>
+        <inertial>
+          <mass value="0.0615752" />
+          <origin xyz="0 0 0" rpy="0 0 0"/>
+          <inertia ixx="9.108e-05" ixy="0" ixz="0" iyy="2.51e-06" iyz="0" izz="8.931e-05" />
+        </inertial>
+      </link>
+      <!-- Camera 2-->
+      <link name="camera2_link">
+        <collision>
+          <origin xyz="0 0 0" rpy="0 0 0"/>
+          <geometry>
+    	       <box size="${camera_length} ${camera_width} ${camera_width}"/>
+          </geometry>
+        </collision>
+        <visual>
+          <origin xyz="0 0 0" rpy="${pi/2} 0 ${pi/2}"/>
+          <geometry>
+    	       <mesh filename="package://ridgeback_yumi_description/meshes/Intel_RealSense_Depth_Camera_D435.STL"/>
+          </geometry>
+          <material name="red"/>
+        </visual>
+        <inertial>
+          <mass value="0.0615752" />
+          <origin xyz="0 0 0" rpy="0 0 0"/>
+          <inertia ixx="9.108e-05" ixy="0" ixz="0" iyy="2.51e-06" iyz="0" izz="8.931e-05" />
+        </inertial>
+      </link>
+      <!-- Camera 3-->
+      <link name="camera3_link">
+        <collision>
+          <origin xyz="0 0 0" rpy="0 0 0"/>
+          <geometry>
+    	       <box size="${camera_length} ${camera_width} ${camera_width}"/>
+          </geometry>
+        </collision>
+        <visual>
+          <origin xyz="0 0 0" rpy="${pi/2} 0 ${pi/2}"/>
+          <geometry>
+    	       <mesh filename="package://ridgeback_yumi_description/meshes/Intel_RealSense_Depth_Camera_D435.STL"/>
+          </geometry>
+          <material name="red"/>
+        </visual>
+        <inertial>
+          <mass value="0.0615752" />
+          <origin xyz="0 0 0" rpy="0 0 0"/>
+          <inertia ixx="9.108e-05" ixy="0" ixz="0" iyy="2.51e-06" iyz="0" izz="8.931e-05" />
+        </inertial>
+      </link>
+        <!-- generate an optical frame http://www.ros.org/reps/rep-0103.html#suffix-frames
+      so that ros and opencv can operate on the camera frame correctly -->
+    <joint name="camera_optical_joint_1" type="fixed">
+    <!-- these values have to be these values otherwise the gazebo camera image
+        won't be aligned properly with the frame it is supposedly originating from -->
     <origin xyz="0 0 0" rpy="${-pi/2} 0 ${-pi/2}"/>
-    <parent link="camera_link_1"/>
+    <parent link="camera1_link"/>
     <child link="camera_link_optical_1"/>
   </joint>
   <link name="camera_link_optical_1">
   </link>
+  <!-- generate an optical frame http://www.ros.org/reps/rep-0103.html#suffix-frames
+      so that ros and opencv can operate on the camera frame correctly -->
   <joint name="camera_optical_joint_2" type="fixed">
+    <!-- these values have to be these values otherwise the gazebo camera image
+        won't be aligned properly with the frame it is supposedly originating from -->
     <origin xyz="0 0 0" rpy="${-pi/2} 0 ${-pi/2}"/>
-    <parent link="camera_link_2"/>
+    <parent link="camera2_link"/>
     <child link="camera_link_optical_2"/>
   </joint>
   <link name="camera_link_optical_2">
   </link>
+  <!-- generate an optical frame http://www.ros.org/reps/rep-0103.html#suffix-frames
+      so that ros and opencv can operate on the camera frame correctly -->
   <joint name="camera_optical_joint_3" type="fixed">
+    <!-- these values have to be these values otherwise the gazebo camera image
+        won't be aligned properly with the frame it is supposedly originating from -->
     <origin xyz="0 0 0" rpy="${-pi/2} 0 ${-pi/2}"/>
-    <parent link="camera_link_3"/>
+    <parent link="camera3_link"/>
     <child link="camera_link_optical_3"/>
   </joint>
   <link name="camera_link_optical_3">
-  </link>
+</link>
 </robot>
